File: Hardware/RC Transmitter.kicad_pcb (KiCad board)
At the start: 4 copper layers, 100 x 76 mm, 83 parts, among them J1 XT60PW-F_C428722, J2 HX25418-3WA, J3 Conn_01x04, J4 BWSMA-KWE-Z001, J5 Conn_02x04_Odd_Even, J6 Conn_02x04_Odd_Even, SW1 SS-12D11G5R, SW2 RKJXV1224005, SW3 RKJXV1224005, SW4 MT-0-102-C004-N004-RS, SW5 MT-0-102-C004-N004-RS, SW6 2AS3T1A1M2QES, SW7 2AS3T1A1M2QES, SW8 2AS3T1A1M2QES, SW9 2AS3T1A1M2QES, U1 MAX17261xxTD, U2 AMS1117-3.3, U3 BQ25887RGE, U4 W25Q128JVS, U5 RP2040, U6 nRF24L01P, U7 RFX2401C, Y1 12MHz, Y2 16MHz

Commit message: PCB update see journal for more information
Parts:
- removed SW2, SW3: RKJXV1224005, lcsc:SW-TH_RKJXV1224005
- added OLED1: HS91L02W2C01, lcsc:OLED-TH_L38.0-W12.0_HS91L02W2C01, F.Cu at (83.7, 167.1)
- added R18: 5.1kΩ, Resistor_SMD:R_0402_1005Metric_Pad0.72x0.64mm_HandSolder, B.Cu at (77.8, 150.3)
- added R19: 5.1kΩ, Resistor_SMD:R_0402_1005Metric_Pad0.72x0.64mm_HandSolder, B.Cu at (79.5, 168.4)
- added U8: YF16-DFL7.2-B5KO(45-10)B5KO(55)-RG-A22, lcsc:JOYTICK-TH_YF16-DFL7.2-B5KO-45-10-B5KO-55--RG-A22, F.Cu at (73.2, 120.8)
- added U9: YF16-FL7.2-B5KA(45-10)-R-A28, lcsc:JOYTICK-TH_YF16-DFL7.2-B5KO-45-10-B5KO-55--RG-A22, F.Cu at (125.9, 120.1)
- moved R16 20.6 mm to (79.5, 170.9), turned to 180 degrees
- moved C1 5.57 mm to (136.7, 115.7), turned to 0 degrees
- moved C20 0.25 mm to (74.2, 145.9)
Connections:
- net /SCL renamed /SCL0
- R16 pad 1: /SDA -> /SDA1
- U1 pad 13: /SDA -> /SDA0
- U3 pad 4: /SDA -> /SDA0
- U5 pad 4: unconnected-(U5-GPIO2-Pad4) -> /SDA1
- U5 pad 5: unconnected-(U5-GPIO3-Pad5) -> /SCL1
- U5 pad 6: /SDA -> /SDA0
Routing:
- net /SDA0: track 0.00 -> 115.5 mm, vias 0 -> 3
- net /SDA: track 114.8 -> 0.00 mm, vias 3 -> 0
- net /BUTTON1: track 73.7 -> 0.00 mm, vias 2 -> 0
- net /SDA1: track 0.00 -> 57.4 mm, vias 0 -> 1
- net /SCL1: track 0.00 -> 57.4 mm, vias 0 -> 1
- net /BUTTON0: track 38.2 -> 0.00 mm
- net +3V3: track 114.3 -> 122.4 mm
- net GND: track 259.5 -> 264.8 mm
- net /AXIS3: track 85.2 -> 80.9 mm
- net /AXIS0: track 48.5 -> 44.8 mm
- net /AXIS1: track 55.7 -> 52.8 mm
- net /UART_RX: track 53.4 -> 52.5 mm
Other:
- outline, holes or cut-outs redrawn

Commit message: PCB upadte
Parts:
- added J7: Conn_01x03, Connector_Wire:SolderWire-0.75sqmm_1x03_P7mm_D1.25mm_OD3.5mm, F.Cu at (100.8, 153.7)
- added JP2: SolderJumper_2_Open, Jumper:SolderJumper-2_P1.3mm_Open_RoundedPad1.0x1.5mm, B.Cu at (107.8, 158.9)
- added R20: 10KΩ, Resistor_SMD:R_0402_1005Metric_Pad0.72x0.64mm_HandSolder, B.Cu at (63.0, 155.7)
- added TP1: TestPoint, TestPoint:TestPoint_Pad_D2.5mm, B.Cu at (144.9, 107.9)
- added TP2: TestPoint, TestPoint:TestPoint_Pad_D2.5mm, B.Cu at (124.6, 156.2)
- added TP3: TestPoint, TestPoint:TestPoint_Pad_D2.5mm, B.Cu at (70.5, 105.0)
- added TP4: TestPoint, TestPoint:TestPoint_Pad_D2.5mm, B.Cu at (76.2, 105.0)
- added TP5: TestPoint, TestPoint:TestPoint_Pad_D2.5mm, B.Cu at (139.8, 107.9)
- moved C10 0.50 mm to (67.8, 157.4)
- moved C11 0.48 mm to (66.2, 155.1)
- moved C15 0.48 mm to (67.3, 155.1)
Connections:
- U5 pad 15: /BUTTON0 -> unconnected-(U5-GPIO12-Pad15)
- U5 pad 16: /BUTTON1 -> unconnected-(U5-GPIO13-Pad16)
- U5 pad 19: unconnected-(U5-TESTEN-Pad19) -> GND
- U5 pad 24: unconnected-(U5-SWCLK-Pad24) -> /SWCLK
- U5 pad 25: unconnected-(U5-SWD-Pad25) -> /SWD
- U5 pad 26: unconnected-(U5-RUN-Pad26) -> /RUN
- U5 pad 56: unconnected-(U5-QSPI_SS-Pad56) -> Net-(U4-~{CS})
- U9 pad 2: /AXIS3 -> /AXIS2
- U9 pad 5: /AXIS2 -> /AXIS3
Routing:
- net GND: track 264.8 -> 355.6 mm
- net /SWD: track 0.00 -> 62.7 mm
- net /RUN: track 0.00 -> 57.6 mm
- net /SWCLK: track 0.00 -> 45.8 mm
- net Net-(U4-~{CS}): track 7.13 -> 31.8 mm
- net +3V3: track 122.4 -> 139.6 mm, vias 14 -> 15
- net VBUS: track 172.5 -> 177.8 mm, vias 3 -> 4
- net +BATT: track 126.4 -> 130.4 mm
- net VDD: track 10.3 -> 14.2 mm
- net /AXIS3: track 80.9 -> 84.7 mm
- net /AXIS2: track 115.3 -> 114.6 mm
Other:
- outline, holes or cut-outs redrawn
- board text added: "+BATT"
- board text added: "3V3"
- board text added: "CHARGER"
- board text added: "FUEL GAUGE"
- board text added: "GND"
- board text added: "OLED DISPLAY"
- board text added: "PROG"
- board text added: "RESET"
- board text added: "RP2040"
- board text added: "SWCLK"
- board text added: "SWD"
- board text added: "VBUS"
- board text added: "VDD"
