File: Hardware/RC Transmitter.kicad_sch (KiCad schematic)
At the start: 85 parts, among them J1 XT60PW-F_C428722, J2 HX25418-3WA, J3 Conn_01x04, J4 BWSMA-KWE-Z001, J5 Conn_02x04_Odd_Even, J6 Conn_02x04_Odd_Even, SW1 SS-12D11G5R, SW2 RKJXV1224005, SW3 RKJXV1224005, SW4 MT-0-102-C004-N004-RS, SW5 MT-0-102-C004-N004-RS, SW6 2AS3T1A1M2QES, SW7 2AS3T1A1M2QES, SW8 2AS3T1A1M2QES, SW9 2AS3T1A1M2QES, U1 MAX17261xxTD, U2 AMS1117-3.3, U3 BQ25887RGE, U4 W25Q128JVS, U5 RP2040, U6 nRF24L01P, U7 RFX2401C, Y1 12MHz, Y2 16MHz

Commit message: PCB update see journal for more information
Parts:
- removed SW2, SW3: RKJXV1224005, lcsc:SW-TH_RKJXV1224005, symbol lcsc:RKJXV1224005
- added OLED1: HS91L02W2C01, lcsc:OLED-TH_L38.0-W12.0_HS91L02W2C01, symbol lcsc:HS91L02W2C01
- added U8: YF16-DFL7.2-B5KO(45-10)B5KO(55)-RG-A22, lcsc:JOYTICK-TH_YF16-DFL7.2-B5KO-45-10-B5KO-55--RG-A22, symbol lcsc:YF16-DFL7.2-B5KO(45-10)B5KO(55)-RG-A22
- added U9: YF16-FL7.2-B5KA(45-10)-R-A28, lcsc:JOYTICK-TH_YF16-DFL7.2-B5KO-45-10-B5KO-55--RG-A22, symbol lcsc:YF16-DFL7.2-B5KO(45-10)B5KO(55)-RG-A22
Connections:
- net +3V3: now also OLED1.3 (SCL), U8.3, U8.6, U9.3, U9.6
- net AXIS0: now also U8.5
- net AXIS1: now also U8.2
- net AXIS2: now also U9.5
- net AXIS3: now also U9.2
- net EP: now also OLED1.4 (SDA), U8.1, U8.10 (shell), U8.4, U8.7 (shell), U8.8 (shell), U8.9 (shell), U9.1, U9.10 (shell), U9.4, U9.7 (shell), U9.8 (shell), U9.9 (shell)
- net SCL0: now also U3.5 (SCL)
- net SCL1: now also OLED1.2 (VCC); no longer U3.5 (SCL)
- net SDA0: now also U3.4 (SDA)
- net SDA1: now also OLED1.1 (GND); no longer U3.4 (SDA)
- net BUTTON0: no longer names the net of U5.15 (GPIO12)
- net BUTTON1: no longer names the net of U5.16 (GPIO13)
Other:
- note added: "DISPLAY"

Commit message: PCB upadte
Parts:
- added J7: Conn_01x03, Connector_Wire:SolderWire-0.75sqmm_1x03_P7mm_D1.25mm_OD3.5mm, symbol Connector_Generic:Conn_01x03
- added JP2: SolderJumper_2_Open, Jumper:SolderJumper-2_P1.3mm_Open_RoundedPad1.0x1.5mm, symbol Jumper:SolderJumper_2_Open
- added R20: 10KΩ, Resistor_SMD:R_0402_1005Metric_Pad0.72x0.64mm_HandSolder, symbol Device:R
- added TP1, TP2, TP3, TP4, TP5: TestPoint, TestPoint:TestPoint_Pad_D2.5mm, symbol Connector:TestPoint
Connections:
- net +3V3: now also R20.1, TP1.1
- net +BATT: now also TP2.1
- net AXIS2: now also U9.2; no longer U9.5
- net AXIS3: now also U9.5; no longer U9.2
- net EP: now also U5.19 (TESTEN), J7.2 (Pin_2), JP2.2 (B), TP3.1
- net VBUS: now also TP4.1
- net VDD: now also TP5.1
- net at R10.1, R11.1, U4.1 (~{CS}): now also U5.56 (QSPI_SS)
- net SWCLK: now reaches U5.24 (SWCLK)
- net SWCLK: now also J7.1 (Pin_1)
- net SWD: now reaches U5.25 (SWD)
- net SWD: now also J7.3 (Pin_3)
- net RUN: now reaches U5.26 (RUN)
- net RUN: now also JP2.1 (A), R20.2
Other:
- note added: "DEBUG OPTIONS"
- moved on the sheet: JP1, R10, R11
